Commit message: Add first version of mock fiducial detector
Added mock fiducial detector node. Modified block and goal URDF
to have mock names for fiducial frames. Added planner to tabletop
launch file. Added mock fiducial detector to mock launch file.

File: urdf/block.xacro (robot description, xacro)
@@ -28,5 +28,5 @@
   </link>
   <!-- The fiducial position -->
-  <link name="block">
+  <link name="mock_block">
     <visual>
       <origin xyz="${-fiducial_thickness/2} 0 0" rpy="0 0 0" />
@@ -39,5 +39,5 @@
   <joint name="block_shape_to_block" type="fixed">
     <parent link="block_shape" />
-    <child link="block" />
+    <child link="mock_block" />
     <origin xyz="${block_side/2} 0 ${block_side - fiducial_size/2}" />
   </joint>

File: urdf/goal.xacro (robot description, xacro)
@@ -43,5 +43,5 @@
   </joint>
   <!-- The goal fiducial -->
-  <link name="goal">
+  <link name="mock_goal">
     <visual>
       <origin xyz="${-fiducial_thickness} 0 0" rpy="0 0 0" />
@@ -54,5 +54,5 @@
   <joint name="goal_back_to_goal" type="fixed">
     <parent link="goal_back" />
-    <child link="goal" />
+    <child link="mock_goal" />
     <origin xyz="0 0 ${fiducial_height}" rpy="0 0 ${pi}" />
   </joint>
